Commit message: implement urdf visualization in rviz

File: cartpole_description/robot/urdf/robot.urdf (robot description, URDF)
Before this commit: robot cartpole_robot, 3 links, 2 joints
Links:
- removed link rail
- added link axis; collision mesh filename=package://cartpole_description/rail.stl; collision mesh filename=package://cartpole_description/stand.stl
- link cart: mass 0.984703 -> None; geometry collision mesh filename=package://cartpole_description/cart.stl; visual mesh filename=package://cartpole_description/cart.stl
- link pole: mass 0.0254927 -> None; geometry collision mesh filename=package://cartpole_description/pole.stl; collision mesh filename=package://cartpole_description/weight.stl
Joints:
- joint slider_cart: parent rail -> axis

Commit message: tweak cartpole_description setup, add documentation

File: cartpole_description/robot/urdf/robot.urdf (robot description, URDF)
Before this commit: robot cartpole_robot, 3 links, 2 joints
Links:
- removed link axis
- added link rail; collision mesh filename=package://cartpole_description/meshes/rail.stl; collision mesh filename=package://cartpole_description/meshes/stand.stl
- link cart: geometry collision mesh filename=package://cartpole_description/meshes/cart.stl; visual mesh filename=package://cartpole_description/meshes/cart.stl
- link pole: geometry collision mesh filename=package://cartpole_description/meshes/pole.stl; collision mesh filename=package://cartpole_description/meshes/weight.stl
Joints:
- joint slider_cart: parent axis -> rail

Commit message: tweak teleop

File: cartpole_description/robot/urdf/robot.urdf (robot description, URDF)
Before this commit: robot cartpole_robot, 3 links, 2 joints
Links:
- link cart: mass None -> 1; geometry collision mesh filename=meshes/cart.stl; visual mesh filename=meshes/cart.stl
- link pole: mass None -> 1; geometry collision mesh filename=meshes/pole.stl; collision mesh filename=meshes/weight.stl
- link rail: mass None -> 0; geometry collision mesh filename=meshes/rail.stl; visual mesh filename=meshes/rail.stl
Joints:
- joint revolute_pole: limit effort=1 velocity=20 -> effort=100 velocity=20
- joint slider_cart: limit lower=-0.42 upper=0.42 effort=1 velocity=20 -> lower=-0.42 upper=0.42 effort=100 velocity=20
