Commit message: add bringup, rearrange desc package

File: cartpole_description/urdf/robot.urdf (robot description, URDF)
Before this commit: robot cartpole_robot, 3 links, 2 joints
Links:
- removed link rail
- added link base_link, mass 0; collision mesh filename=package://cartpole_description/meshes/rail.stl; visual mesh filename=package://cartpole_description/meshes/rail.stl
- link cart: geometry collision mesh filename=package://cartpole_description/meshes/cart.stl; visual mesh filename=package://cartpole_description/meshes/cart.stl
- link pole: geometry collision mesh filename=package://cartpole_description/meshes/pole.stl; collision mesh filename=package://cartpole_description/meshes/weight.stl
Joints:
- joint slider_cart: parent rail -> base_link
